File: HW/KiCAD/STM32G4 V1.0/connector.kicad_sch (KiCad schematic)
At the start: 9 parts, among them J1 Conn_01x14, J4 Conn_01x11, J7 Conn_01x06

Commit message: sch pdf add
Other:
- title: (none) -> STM32G4 MAZE V1.0
Changed lines of the file:
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@@
   (paper "A4")
   (title_block
+    (title "STM32G4 MAZE V1.0")
     (date "2023-08-16")
     (company "MAZE")
