File: HW/KiCAD/STM32G4 V1.0/microcontroller.kicad_sch (KiCad schematic)
At the start: 20 parts, among them U1 STM32G4xxV, Y1 ECS-200-9-33B-CTP-TR, Y2 ECS-.327-9-34B-C-TR

Commit message: sch pdf add
Other:
- title: (none) -> STM32G4 MAZE V1.0
Changed lines of the file:
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@@
   (paper "A4")
   (title_block
+    (title "STM32G4 MAZE V1.0")
     (date "2023-08-16")
     (company "MAZE")
